Commit message: make change to support two wheel velocity only configuration

File: mecanumbot_description/urdf/mecanumbot.urdf (robot description, URDF)
Before this commit: robot mecanumbot, 6 links, 5 joints
Links:
- removed link fl_wheel_link
- removed link fr_wheel_link
- removed link rl_wheel_link
- removed link rr_wheel_link
- added link l_wheel_link, mass ${wheel_mass}; collision box size=${wheel_radius*2} ${wheel_width} ${wheel_radius*2}; visual box size=${wheel_radius*2} ${wheel_width} ${wheel_radius*2}
- added link r_wheel_link, mass ${wheel_mass}; collision box size=${wheel_radius*2} ${wheel_width} ${wheel_radius*2}; visual box size=${wheel_radius*2} ${wheel_width} ${wheel_radius*2}
Joints:
- removed joint fl_wheel_joint
- removed joint fr_wheel_joint
- removed joint rl_wheel_joint
- removed joint rr_wheel_joint
- added joint l_wheel_joint: type continuous, parent base_link, child l_wheel_link, origin xyz=0.19 0.23 ${wheel_offset_z} rpy=0 0 0
- added joint r_wheel_joint: type continuous, parent base_link, child r_wheel_link, origin xyz=0.19 -0.23 ${wheel_offset_z} rpy=0 0 0
